File: Schaltung/Schaltung.sch (KiCad schematic (older format))
At the start: 23 parts, among them J1 Barrel_Jack, J2 double WS2812b Connector, J3 new_Firmware, Q1 2N2222, Q2 SMP60N03, SW1 Bootlader, SW2 Reset, U1 HT7833, U2 ESP-12E

Commit message: change mosfet to IRLZ44N
Parts:
- Q2: value SMP60N03 -> IRLZ44N
Changed lines of the file:
@@
 P 2500 3600
 F 0 "Q2" H 2750 3675 50  0000 L CNN
-F 1 "SMP60N03" H 2750 3600 50  0000 L CNN
+F 1 "IRLZ44N" H 2750 3600 50  0000 L CNN
 F 2 "TO_SOT_Packages_THT:TO-220_Vertical" H 2750 3525 50  0001 L CIN
 F 3 "" H 2500 3600 50  0001 L CNN

Commit message: add IR Receiver
Parts:
- removed D2: D_Schottky, symbol D_Schottky
- added U3: TSOP45xx, Opto-Devices:IRReceiver_Vishay_MOLD-3pin, symbol TSOP45xx
Connections:
- net +3V3: now also J3.1 (Pin_1), R4.2, R5.2, R8.1, U2.8 (VCC), U3.3 (Vs)
- net GND: now also U3.2 (GND)
- net at U2.10 (GPIO15): now also U3.1 (OUT)
Changed lines of the file:
@@
 L +3.3V #PWR8
 U 1 1 5A77760D
-P 4500 2450
-F 0 "#PWR8" H 4500 2300 50  0001 C CNN
-F 1 "+3.3V" H 4500 2590 50  0000 C CNN
-F 2 "" H 4500 2450 50  0001 C CNN
-F 3 "" H 4500 2450 50  0001 C CNN
-	1    4500 2450
+P 4500 2750
+F 0 "#PWR8" H 4500 2600 50  0001 C CNN
+F 1 "+3.3V" H 4500 2890 50  0000 C CNN
+F 2 "" H 4500 2750 50  0001 C CNN
+F 3 "" H 4500 2750 50  0001 C CNN
+	1    4500 2750
 	-1   0    0    -1
 $EndComp
@@
 $EndComp
 $Comp
-L D_Schottky D2
-U 1 1 5A77EFB0
-P 4500 2600
-F 0 "D2" H 4500 2700 50  0000 C CNN
-F 1 "D_Schottky" H 4500 2500 50  0000 C CNN
-F 2 "" H 4500 2600 50  0001 C CNN
-F 3 "" H 4500 2600 50  0001 C CNN
-	1    4500 2600
-	0    -1   -1   0
-$EndComp
-$Comp
 L Q_PNP_CBE Q1
 U 1 1 5A7A4EB9
@@
 	4450 3150 4900 3150
 Wire Wire Line
-	7600 2950 6700 2950
+	6700 2950 7750 2950
 Wire Wire Line
 	7600 2950 7600 3750
@@
 	4150 3550 4000 3550
 Connection ~ 4000 3550
+$Comp
+L TSOP45xx U3
+U 1 1 5A7A6426
+P 8150 2750
+F 0 "U3" H 7750 3050 50  0000 L CNN
+F 1 "TSOP45xx" H 7750 2450 50  0000 L CNN
+F 2 "Opto-Devices:IRReceiver_Vishay_MOLD-3pin" H 8100 2375 50  0001 C CNN
+F 3 "" H 8800 3050 50  0001 C CNN
+	1    8150 2750
+	-1   0    0    -1
+$EndComp
+$Comp
+L +3.3V #PWR?
+U 1 1 5A7A6807
+P 7600 2400
+F 0 "#PWR?" H 7600 2250 50  0001 C CNN
+F 1 "+3.3V" H 7600 2540 50  0000 C CNN
+F 2 "" H 7600 2400 50  0001 C CNN
+F 3 "" H 7600 2400 50  0001 C CNN
+	1    7600 2400
+	-1   0    0    -1
+$EndComp
+Wire Wire Line
+	7750 2550 7600 2550
+Wire Wire Line
+	7600 2550 7600 2400
+Connection ~ 7600 2950
+Wire Wire Line
+	6700 3050 6800 3050
+Wire Wire Line
+	6800 3050 6800 2750
+Wire Wire Line
+	6800 2750 7750 2750
 $EndSCHEMATC
